Commit message: config for park_dataset with odom/imu in navsat

File: launch/include/config/robot.urdf.xacro (robot description, xacro)
@@ -27,3 +27,9 @@
     <origin xyz="0 0 0" rpy="0 0 0" />
   </joint>
+  <link name="odom_imu"> </link>
+  <joint name="odomimu_joint" type="fixed">
+    <parent link="chassis_link" />
+    <child link="odom_imu" />
+    <origin xyz="0 0 0" rpy="0 0 0" />
+  </joint>
 </robot>
